File: Placa do elevador controlador femea/Placa do elevador.kicad_pcb (KiCad board)
At the start: 2 copper layers, 108.5 x 84.8 mm, 7 parts, among them J1 DB25_Female, J2 Conn_01x04, J3 Conn_01x04, J4 Conn_01x04, J5 Conn_01x04, J6 Conn_01x04, J7 Conn_01x04

Commit message: Mudando de nome e atualizando os perfis
Parts:
- moved J1 26.4 mm to (157.0, 75.9), turned to 180 degrees
Routing:
- net M1: track 110.6 -> 0.00 mm
- net L2: track 110.5 -> 0.00 mm
- net L6: track 103.6 -> 0.00 mm
- net L4: track 97.1 -> 0.00 mm
- net L5: track 95.5 -> 0.00 mm
- net L3: track 76.2 -> 0.00 mm
- net B1: track 75.6 -> 0.00 mm
- net B4: track 67.4 -> 0.00 mm
- net B2: track 61.9 -> 0.00 mm
- net L1: track 53.2 -> 0.00 mm
- net +5V: track 43.5 -> 0.00 mm
- net +5VA: track 43.2 -> 0.00 mm
- net +12V: track 42.9 -> 0.00 mm
- net B5: track 42.7 -> 0.00 mm
- net B3: track 42.3 -> 0.00 mm
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