File: Placa do elevador controlador femea/Placa do elevador.sch (KiCad schematic (older format))
At the start: 7 parts, among them J1 DB25_Female, J2 Conn_01x04, J3 Conn_01x04, J4 Conn_01x04, J5 Conn_01x04, J6 Conn_01x04, J7 Conn_01x04

Commit message: Mudando de nome e atualizando os perfis
Parts:
- J1: footprint Connector_Dsub:DSUB-25_Female_Horizontal_P2.77x2.84mm_EdgePinOffset14.56mm_Housed_MountingHolesOffset8.20mm -> Connector_Dsub:DSUB-25_Female_Horizontal_P2.77x2.84mm_EdgePinOffset14.56mm_Housed_MountingHolesOffset15.98mm
Changed lines of the file:
@@
 EESchema Schematic File Version 4
+LIBS:Placa do elevador-cache
 EELAYER 26 0
 EELAYER END
@@
 F 0 "J1" H 2570 4117 50  0000 C CNN
 F 1 "DB25_Female" H 2570 4026 50  0000 C CNN
-F 2 "Connector_Dsub:DSUB-25_Female_Horizontal_P2.77x2.84mm_EdgePinOffset14.56mm_Housed_MountingHolesOffset8.20mm" H 2650 2625 50  0001 C CNN
+F 2 "Connector_Dsub:DSUB-25_Female_Horizontal_P2.77x2.84mm_EdgePinOffset14.56mm_Housed_MountingHolesOffset15.98mm" H 2650 2625 50  0001 C CNN
 F 3 " ~" H 2650 2625 50  0001 C CNN
 	1    2650 2625
